File: src_files/_autosave-ad_power_device.sch (KiCad schematic (older format))
At the start: 34 parts, among them J1 SPEAKER, J2 5622-6309-ML, Q1 DTC143ZEBTL, Q2 DTC143ZEBTL, U7 QUECTEL_L70-RL

Commit message: update NFC, 5G, GPS__left LiPo charger+screen changes
Other:
- note added: "I2C_PULLUP"
- note added: "NFC_IC_VS1797SM"
- moved on the sheet: R?
Changed lines of the file:
@@
 TO HDMI
 $Sheet
-S 1775 4800 1675 525
+S 775  4750 1675 525
 U 61B4DD57
 F0 "OTHER_POWER" 50
@@
 Wire Wire Line
 	8100 2475 8250 2475
-Text GLabel 1150 8100 1    39   Input ~ 0
+Text GLabel 1125 7900 1    39   Input ~ 0
 VCC3V3_PMU
 $Comp
 L Device:R_US R?
 U 1 1 661B72AA
-P 950 8350
-F 0 "R?" H 825 8275 50  0000 C CNN
-F 1 "4.7K" H 836 8350 50  0000 C CNN
-F 2 "Resistor_SMD:R_0402_1005Metric" V 990 8340 50  0001 C CNN
-F 3 "~" H 950 8350 50  0001 C CNN
-	1    950  8350
+P 925 8150
+F 0 "R?" H 800 8075 50  0000 C CNN
+F 1 "4.7K" H 811 8150 50  0000 C CNN
+F 2 "Resistor_SMD:R_0402_1005Metric" V 965 8140 50  0001 C CNN
+F 3 "~" H 925 8150 50  0001 C CNN
+	1    925  8150
 	-1   0    0    1
 $EndComp
@@
 L Device:R_US R?
 U 1 1 662413A3
-P 1325 8350
-F 0 "R?" H 1200 8275 50  0000 C CNN
-F 1 "4.7K" H 1211 8350 50  0000 C CNN
-F 2 "Resistor_SMD:R_0402_1005Metric" V 1365 8340 50  0001 C CNN
-F 3 "~" H 1325 8350 50  0001 C CNN
-	1    1325 8350
+P 1300 8150
+F 0 "R?" H 1175 8075 50  0000 C CNN
+F 1 "4.7K" H 1186 8150 50  0000 C CNN
+F 2 "Resistor_SMD:R_0402_1005Metric" V 1340 8140 50  0001 C CNN
+F 3 "~" H 1300 8150 50  0001 C CNN
+	1    1300 8150
 	-1   0    0    1
 $EndComp
 Wire Wire Line
-	950  8200 950  8150
-Wire Wire Line
-	950  8150 1150 8150
-Wire Wire Line
-	1150 8150 1150 8100
-Wire Wire Line
-	1150 8150 1325 8150
-Wire Wire Line
-	1325 8150 1325 8200
-Connection ~ 1150 8150
-Text Label 950  8600 3    50   ~ 0
+	925  8000 925  7950
+Wire Wire Line
+	925  7950 1125 7950
+Wire Wire Line
+	1125 7950 1125 7900
+Wire Wire Line
+	1125 7950 1300 7950
+Wire Wire Line
+	1300 7950 1300 8000
+Connection ~ 1125 7950
+Text Label 925  8400 3    50   ~ 0
 NFC_SDA
-Text Label 1325 8625 3    50   ~ 0
+Text Label 1300 8425 3    50   ~ 0
 NFC_SCL
 Wire Wire Line
-	950  8500 950  8600
-Wire Wire Line
-	1325 8500 1325 8625
+	925  8300 925  8400
+Wire Wire Line
+	1300 8300 1300 8425
 Wire Wire Line
 	2575 9350 2575 9400
@@
 Wire Notes Line
 	4625 5800 2650 5800
+Wire Notes Line
+	4475 5975 4475 7350
+Wire Notes Line
+	4475 7350 550  7350
+Wire Notes Line
+	550  7350 550  5975
+Wire Notes Line
+	550  5975 4475 5975
+Text Notes 1575 7875 2    39   ~ 0
+I2C_PULLUP
+Text Notes 2725 8925 2    39   ~ 0
+NFC_IC_VS1797SM
+Wire Notes Line
+	575  7425 1675 7425
+Wire Notes Line
+	1675 7425 1675 8800
+Wire Notes Line
+	1675 8800 575  8800
+Wire Notes Line
+	575  8800 575  7425
+Wire Notes Line
+	600  8850 3950 8850
+Wire Notes Line
+	3950 8850 3950 11100
+Wire Notes Line
+	3950 11100 600  11100
+Wire Notes Line
+	600  11100 600  8850
 $EndSCHEMATC
