File: src_files/OTHER_POWER.sch (KiCad schematic (older format))
At the start: 0 parts

Commit message: schematic capture complete
Parts:
- added C220, C221, C270, C280, C281, C282: 10uF, Capacitor_SMD:C_0402_1005Metric, symbol Device:C_Small
- added C222, C223, C224, C225: 22uF, Capacitor_SMD:C_0402_1005Metric, symbol Device:C_Small
- added C271, C278: 100nF, Capacitor_SMD:C_0402_1005Metric, symbol Device:C_Small
- added C272: 100NF, Capacitor_SMD:C_0402_1005Metric, symbol Device:C_Small
- added C273: 2.2uF, Capacitor_SMD:C_0402_1005Metric, symbol Device:C_Small
- added C274: 39nF, Capacitor_SMD:C_0402_1005Metric, symbol Device:C_Small
- added C275: 82pF, Capacitor_SMD:C_0402_1005Metric, symbol Device:C_Small
- added C276, C277: 22uF_16V, Capacitor_SMD:C_0603_1608Metric, symbol Device:C_Small
- added C279: 4.7uF, Capacitor_SMD:C_0402_1005Metric, symbol Device:C_Small
- added D18: SS56, greencharge-footprints:SMAG, symbol Device:D
- added IC1: TPS62867RQYR, greencharge-footprints:TPS62865RQYR, symbol GCL_Integrated-Circuits:TPS62867RQYR
- added IC2: TPS61288RQQR, greencharge-footprints:TPS61288RQQR, symbol GCL_Integrated-Circuits:TPS61288RQQR
- added L11: RLF12560T2R7N110, greencharge-footprints:RLF12560T2R7N110, symbol Device:L
- added L12: IHLP1212AEERR22M11, greencharge-footprints:INDPM3630X150N, symbol SamacSys_Parts:IHLP1212AEERR22M11
- added L14: 2.2uH, greencharge-footprints:WPN4020H2R2MT, symbol OLIMEX_RCL:INDUCTOR_SMALL
- added R100: 931K, Resistor_SMD:R_0402_1005Metric, symbol Device:R_US
- added R101: 48.7K, Resistor_SMD:R_0402_1005Metric, symbol Device:R_US
- added R102: 20K, Resistor_SMD:R_0402_1005Metric, symbol Device:R_US
- added R103: 475K, Resistor_SMD:R_0402_1005Metric, symbol Device:R_US
- added R104, R105, R76: 100K, Resistor_SMD:R_0402_1005Metric, symbol Device:R_US
- added R27: 34K, Resistor_SMD:R_0402_1005Metric, symbol Device:R_US
- added R77: 205K, Resistor_SMD:R_0402_1005Metric, symbol Device:R_US
- added R78: 6.8K_1%, Resistor_SMD:R_0402_1005Metric, symbol Device:R_US
- added TP12: VDD_CPU, TestPoint:TestPoint_Pad_D1.0mm, symbol Connector:TestPoint
- added TP13: 3V3, TestPoint:TestPoint_Pad_D1.0mm, symbol Connector:TestPoint
- added TP14: 12V, TestPoint:TestPoint_Pad_D1.0mm, symbol Connector:TestPoint
- added TP15: VCC3V3_EXT, TestPoint:TestPoint_Pad_D1.0mm, symbol Connector:TestPoint
- added U17: SY6280AAAC, Package_TO_SOT_SMD:SOT-23-5, symbol GCL_Integrated-Circuits:SY6280AAAC
- added U6: TLV62569PDDCR, Package_TO_SOT_SMD:SOT-23-6, symbol Regulator_Switching:TLV62569DDC
Connections:
- new net: IC2.1 (FB_1), IC2.12 (FB_1), R100.2, R101.1
- new net: C273.1, IC2.11 (VCC)
- new net: C275.1, IC2.2 (COMP), R27.1
- new net: C272.1, IC2.4 (SW_1), IC2.9 (SW_1), L11.2
- new net: C272.2, IC2.8 (BST)
- new net: C274.1, R27.2
- new net: C278.1, R102.1, U6.1 (EN)
- new net: L14.1, U6.3 (SW)
- new net: R103.1, U6.5 (PG)
- new net: R104.2, R105.1, U6.6 (FB)
- new net: IC1.5 (PG), R76.1
- new net: IC1.6 (VSET/MODE), R77.1
- new net: IC1.7 (SW), L12.1
- new net: R78.1, U17.3 (OCB)
- new net +12V: C276.1, C277.1, IC2.14 (VOUT_1), IC2.5 (VOUT_1), R100.1, TP14.1
- new net +3V3: C222.1, C223.1, C224.1, C270.1, C271.1, C279.1, IC1.8 (VOS), IC1.9 (FB), IC2.15 (VIN_1), IC2.6 (EN), IC2.7 (VIN_1), L11.1, L12.2, R103.2, TP13.1, U17.5 (1N), U6.4 (VIN)
- new net +5V: C220.1, C221.1, D18.1 (K), IC1.3 (VIN), IC1.4 (EN), R76.2
- new net GND: C220.2, C221.2, C222.2, C223.2, C224.2, C225.2, C270.2, C271.2, C273.2, C274.2, C275.2, C276.2, C277.2, C278.2, C279.2, C280.2, C281.2, C282.2, IC1.1 (AGND), IC1.2 (PGND), IC2.10 (AGND), IC2.13 (PGND_2), IC2.3 (PGND_1), R101.2, R105.2, R77.2, R78.2, U17.2 (GND), U6.2 (GND)
- new net PMIC_EXT_EN: U17.4 (EN)
- new net VBAT: D18.2 (A)
- new net VCC3V3_EXT: C225.1, TP15.1, U17.1 (VOUT)
- new net VCC3V3_PMU: R102.2
- new net VDD_CPU: C280.1, C281.1, C282.1, L14.2, R104.1, TP12.1
Other:
- note added: "3.3V TO 1.2V @1A FOR VDD_CPU"
- note added: "3V-5V TO 12V @ 2A"
- note added: "3V3 MAIN SOURCE"
- note added: "5V TO 3.3V @ 5A"
- note added: "OVERCURRENT/SHOERT CIRCUIT PROTECTION"
- note added: "TO SUPPLY EXTERNAL COMPONENTS"
