File: src_files/RK3566_PART_C.sch (KiCad schematic (older format))
At the start: 77 parts, among them J4 3-1734592-0, J5 3-1734592-0, J6 3-1734592-0, U1 RK3566

Commit message: complete update on schematic and all display interfaces
Parts:
- added C190, C297: 100nF, Capacitor_SMD:C_0402_1005Metric, symbol Device:C_Small
- added C204, C205: 10uF, Capacitor_SMD:C_0603_1608Metric, symbol Device:C_Small
- added D2: 1N5819WS, Diode_SMD:D_SOD-323, symbol Device:D
- added D3: ESD5451R-2/TR, greencharge-footprints:DFP1006-2L, symbol Device:D_TVS
- added R46, R60: 2.2K_5%, Resistor_SMD:R_0402_1005Metric, symbol Device:R_US
- added R64: 1K, Resistor_SMD:R_0402_1005Metric, symbol Device:R_US
- added R65: 1KK, Resistor_SMD:R_0402_1005Metric, symbol Device:R_US
- added U9: ZLDO1117G12TA, Package_TO_SOT_SMD:SOT-223-3_TabPin2, symbol Regulator_Linear:LF85_TO220
- Y4: renamed from Y?; value XLH536025_000000I -> ASE-27.000MHZ-LR-T(27MHz)
- gave numbers to parts that had none: 17
Connections:
- net INT is gone; now on net INT_hdmi_to_mipi: U8.J4 (INT)
- net MIPI_DSI_TX1_D3N- is gone; now on net MIPI_DSI_TX1_D3-: U1.AP20 (MIPI_DSI_TX1_D3n)
- net MIPI_DSI_TX1_D3P+ is gone; now on net MIPI_DSI_TX1_D3+: U1.AR20 (MIPI_DSI_TX1_D3p)
- net +1V2: now also C205.1, U9.3 (VO)
- net +3V3: now also C204.1, C297.1, D2.2 (A), U9.1 (VI)
- net GND: now also C190.2, C204.2, C205.2, C297.2, D3.2 (A2), R65.2, U9.2 (GND)
- net HDMI_TX_HPDIN: now also R64.2
- net MCDP_I2C_SCL: now also U8.J5 (I2C_SCL), R60.2; no longer U8.K5 (I2C_SDA)
- net MCDP_I2C_SDA: now also U8.K5 (I2C_SDA), R46.2; no longer U8.J5 (I2C_SCL)
- net MIPI_D1+: now also U8.E9 (MIPI_D1N)
- net MIPI_D1-: now also U8.E10 (MIPI_D1P)
- net VCC5V_HDMI_TX: now also D2.1 (K), D3.1 (A1)
- net VCC_3V3: now reaches U1.1N5 (VCCIO5_1)
- net VCC_3V3: now also U1.1N6 (VCCIO5_2), C190.1
- net TP_RST_L_GPIO0_C5_DISPLAY_THREE: now reaches U1.1P3 (UART7_TX_M1)
- net LCD_BL_PWM10_M0_DISPLAY_THREE: now reaches U1.1P4 (UART7_RX_M)
- net INT_eDP_MIPI: now reaches U1.1U4 (GMAC1_TXCLK_M0)
- net HPD_eDP_mipi: now reaches U1.1V3 (GMAC1_RXCLK_M0)
- net BL_EN_GPIO0_C0_DISPLAY_THREE: now reaches U1.AP3 (UART5_TX_M1)
- net TP_INT_GPIO0_A5_DISPLAY_THREE: now reaches U1.AP4 (PCIE20_PERSTn_M1)
- net GPIO1_C2_u_DISPLAY_THREE: now reaches U1.AP9 (GMAC1_RXD3_M0)
- net LCD_RST_L_GPIO0_C2_DISPLAY_THREE: now reaches U1.AR2 (UART5_RX_M1)
- net LCD_3_ENGPIO1_C3_u_TO_DISPLAY: now reaches U1.AR4 (UART3_RX_M1)
- net INT_hdmi_to_mipi: now reaches U1.AR7 (ETH1_REFCLKO_25M_M0)
- net EDP_TX_D3+: now reaches U1.N37 (EDP_TX_D3p)
- net EDP_TX_D3-: now reaches U1.N38 (EDP_TX_D3n)
- net HDMI_TXDDC_SCL_PORT renamed HDMITX_SCL
- net HDMI_TXDDC_SDA_PORT renamed HDMITX_SDA
- net HDMI_TX_CEC_PORT renamed HDMITX_CEC_M0
- net HDMI_TX_HPD_PORT: no longer names the net of U8.K3 (HPDI)
- net HDMI_TX_HPD_PORT: now also R64.1, R65.1
- net MIPI_DSI_TX1_CLKN- renamed MIPI_DSI_TX1_CLK-
- net MIPI_DSI_TX1_CLKP+ renamed MIPI_DSI_TX1_CLK+
- net MIPI_DSI_TX1_D0N- renamed MIPI_DSI_TX1_D0-
- net MIPI_DSI_TX1_D0P+ renamed MIPI_DSI_TX1_D0+
- net MIPI_DSI_TX1_D1N- renamed MIPI_DSI_TX1_D1-
- net MIPI_DSI_TX1_D1P+ renamed MIPI_DSI_TX1_D1+
- net MIPI_DSI_TX1_D2N- renamed MIPI_DSI_TX1_D2-
- net MIPI_DSI_TX1_D2P+ renamed MIPI_DSI_TX1_D2+
- net UART4_RX: no longer names the net of U1.AP7 (GMAC1_RXD0_M0)
- net UART4_TX: no longer names the net of U1.AR6 (GMAC1_RXD1_M0)
- new net VCC3V3_PMU: R46.1, R60.1
- no-connect marks 33 -> 19
Other:
- note added: "1.2V MCDP SUPPLY"
- note added: "I2C_PULLUP"
- note removed: "TO GPS MODULE"

Commit message: complete update on schematiC + FOOTPRINT
Parts:
- U8: footprint (none) -> greencharge-footprints:TC358779XBG
Changed lines of the file:
@@
 F 0 "U8" H 15675 8525 50  0000 C CNN
 F 1 "TC358779XBG" H 15650 8425 50  0000 C CNN
-F 2 "" H 14550 9350 50  0001 C CNN
+F 2 "greencharge-footprints:TC358779XBG" H 14550 9350 50  0001 C CNN
 F 3 "" H 14550 9350 50  0001 C CNN
 	1    15550 10050
