File: src_files/AP6256_WIFI_BT.sch (KiCad schematic (older format))
At the start: 18 parts, among them J16 U.FL-R-SMT-1(10), U3 AP6256, Y2 37.4MHz_10PPM

Commit message: layout change
Changed lines of the file:
@@
 AR Path="/629B27D4/61E5D3CF" Ref="J16"  Part="1"
 F 0 "J16" H 800 1625 50  0000 L CNN
-F 1 "U.FL-R-SMT-1(10)" H 575 1525 50  0000 L CNN
+F 1 "U.FL-R-SMT-1(10)" H 285 1545 50  0000 L CNN
 F 2 "greencharge-footprints:HRS_U.FL-R-SMT-1(10)" H 825 1350 50  0001 L BNN
 F 3 "" H 825 1350 50  0001 L BNN
