File: src_files/ad_power_device.kicad_pcb (KiCad board)
At the start: 2 copper layers, 75 x 75 mm, 593 parts, among them IC1 TPS62867RQYR, IC2 TPS61288RQQR, IC3 P9038, J13 U.FL-R-SMT-1(10), J14 U.FL-R-SMT-1(10), J16 U.FL-R-SMT-1(10), J2 5622-6309-ML, J3 205957-0271, J4 3-1734592-0, J5 3-1734592-0, J6 3-1734592-0, J7 Conn_01x05_Male, J8 3-1734592-0, J9 SIM8066-6-1-14-01-A_REVA, Q10 DTC143ZEBTL, Q11 IRFR9024NTRPBF, Q12 DTC143ZEBTL, Q6 DTC143ZEBTL, Q7 DTC143ZEBTL, Q8 DTC143ZEBTL, Q9 DTC143ZEBTL, SW1 PWR_ON, SW2 RESET BTN, SW3 RECOVER BTN, U1 RK3566, U10 TC358860XBG, U11 NFC_VS1797SM, U12 TLV71211DBVR, U13 STWLC68, U14 TPS56637RPAR, U15 24AA64T-I/OT, U16 BRCS120N02ZJ, U17 SY6280AAAC, U18 ESD5304D-TP, U19 EG25G, U2 RK809, U20 ESD5304D-TP, U21 SY6912A, U3 AP6256, U4 LPDDR4_32_IS43LQ32128A-062BLI, U5 TLV62569PDDCR, U6 TLV62569PDDCR, U7 TPS63802DLAR, U8 TC358779XBG, U9 ZLDO1117G12TA, Y1 32.768KHz, Y2 37.4MHz_10PPM, Y3 24MHz/10ppm, Y4 ASE-27.000MHZ-LR-T(27MHz), Y5 ASE-27.000MHZ-LR-T(27MHz)

Commit message: layout change
Parts:
- J8: moved to F.Cu
- moved J8 41.3 mm to (51.6, 154.4), turned to 180 degrees
- moved C237 1.25 mm to (48.3, 164.2)
- moved C296 1.25 mm to (62.5, 160.2)
- moved C86 1.25 mm to (48.0, 160.0)
- moved C89 1.25 mm to (48.0, 158.1)
- moved L3 1.25 mm to (61.9, 157.9)
- moved C208 1.25 mm to (56.8, 158.2)
- moved C287 1.25 mm to (56.7, 160.2)
- moved C288 1.25 mm to (59.6, 160.2)
- moved C292 1.25 mm to (59.6, 158.2)
- moved C64 1.25 mm to (61.4, 164.5)
- moved C85 1.25 mm to (44.3, 163.7)
- moved C87 1.25 mm to (50.9, 158.1)
- moved C91 1.25 mm to (47.1, 162.1)
- moved C93 1.25 mm to (50.9, 160.0)
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